File: CheeseBoardCheddar_PCB/CheeseBoardCheddar.sch (KiCad schematic (older format))
At the start: 33 parts, among them P1 USB_Micro, P10 LOGO1, P11 LOGO2, P12 KNOB, P13 LOGO_CHEESE, P2 5V_EXT, P3 SERIAL_HC12, P4 S_SERIAL, P5 NODEMCU_1, P6 NODEMCU_2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

Commit message: Updated PCB with Encoder switch sorted
Parts:
- P1: Supplier 2 (none) -> Farnell; Supplier 2 Cost (none) -> 0.474; Supplier 2 Part No (none) -> 2396171
Connections:
- net +3V3: now also ENC1.2
- net GND: no longer ENC1.2
Other:
- moved on the sheet: DISP1, ENC1, P12, P13, P8

Commit message: Added I2C bus to PCB
Parts:
- added P14: I2C_EXT, REInnovationFootprint:SIL-4_large_pad, symbol CONN_01X04
Connections:
- net 5V_PWR: now also P14.3 (P3)
- net GND: now also P14.4 (P4)
- net LED_WS2811: now also P14.2 (P2)
- net SDA: now also P14.1 (P1)
Changed lines of the file:
@@
 LIBS:contrib
 LIBS:valves
+LIBS:matts_components
 LIBS:CheeseBoardCheddar-cache
 EELAYER 25 0
@@
 NoConn ~ 6500 5050
 $Comp
-L +3.3V #PWR?
+L +3.3V #PWR020
 U 1 1 59C7D210
 P 10500 1850
-F 0 "#PWR?" H 10500 1700 50  0001 C CNN
+F 0 "#PWR020" H 10500 1700 50  0001 C CNN
 F 1 "+3.3V" H 10500 1990 50  0000 C CNN
 F 2 "" H 10500 1850 50  0000 C CNN
@@
 Wire Wire Line
 	10500 1950 10500 1850
+$Comp
+L CONN_01X04 P14
+U 1 1 5A22E883
+P 9450 4600
+F 0 "P14" H 9450 4850 50  0000 C CNN
+F 1 "I2C_EXT" V 9550 4600 50  0000 C CNN
+F 2 "REInnovationFootprint:SIL-4_large_pad" H 9450 4600 50  0001 C CNN
+F 3 "" H 9450 4600 50  0000 C CNN
+	1    9450 4600
+	1    0    0    -1
+$EndComp
+$Comp
+L GND #PWR021
+U 1 1 5A22F1EB
+P 9000 4850
+F 0 "#PWR021" H 9000 4600 50  0001 C CNN
+F 1 "GND" H 9000 4700 50  0000 C CNN
+F 2 "" H 9000 4850 50  0000 C CNN
+F 3 "" H 9000 4850 50  0000 C CNN
+	1    9000 4850
+	1    0    0    -1
+$EndComp
+Text HLabel 8950 4450 0    60   Input ~ 0
+SDA
+Text HLabel 8950 4550 0    60   Input ~ 0
+SCL
+Wire Wire Line
+	9250 4650 8550 4650
+Wire Wire Line
+	9000 4850 9000 4750
+Wire Wire Line
+	9000 4750 9250 4750
+Wire Wire Line
+	8950 4550 9250 4550
+Wire Wire Line
+	8950 4450 9250 4450
+Text HLabel 8550 4650 0    60   Input ~ 0
+5V_PWR
 $EndSCHEMATC

Commit message: Update of instructions
Parts:
- removed P14: I2C_EXT, REInnovationFootprint:SIL-4_large_pad, symbol CONN_01X04
- added P14: I2C_EXT, matts_components:SIL-5_large_pads_marker, symbol CONN_01X05
Connections:
- net +3V3: now also P14.1 (P1)
- net 5V_PWR: now also P14.4 (P4)
- net GND: now also P14.5 (P5)
- net LED_WS2811: now also P14.3 (P3)
- net SDA: now also P14.2 (P2)
Changed lines of the file:
@@
 LIBS:contrib
 LIBS:valves
-LIBS:matts_components
 LIBS:CheeseBoardCheddar-cache
 EELAYER 25 0
@@
 	10500 1950 10500 1850
 $Comp
-L CONN_01X04 P14
-U 1 1 5A22E883
-P 9450 4600
-F 0 "P14" H 9450 4850 50  0000 C CNN
-F 1 "I2C_EXT" V 9550 4600 50  0000 C CNN
-F 2 "REInnovationFootprint:SIL-4_large_pad" H 9450 4600 50  0001 C CNN
-F 3 "" H 9450 4600 50  0000 C CNN
-	1    9450 4600
-	1    0    0    -1
-$EndComp
-$Comp
 L GND #PWR021
 U 1 1 5A22F1EB
@@
 Text HLabel 8550 4650 0    60   Input ~ 0
 5V_PWR
+$Comp
+L CONN_01X05 P14
+U 1 1 5A29A719
+P 9450 4550
+F 0 "P14" H 9450 4850 50  0000 C CNN
+F 1 "I2C_EXT" V 9550 4550 50  0000 C CNN
+F 2 "matts_components:SIL-5_large_pads_marker" H 9450 4550 50  0001 C CNN
+F 3 "" H 9450 4550 50  0000 C CNN
+	1    9450 4550
+	1    0    0    -1
+$EndComp
+$Comp
+L +3.3V #PWR022
+U 1 1 5A29A923
+P 9050 4300
+F 0 "#PWR022" H 9050 4150 50  0001 C CNN
+F 1 "+3.3V" H 9050 4440 50  0000 C CNN
+F 2 "" H 9050 4300 50  0000 C CNN
+F 3 "" H 9050 4300 50  0000 C CNN
+	1    9050 4300
+	1    0    0    -1
+$EndComp
+Wire Wire Line
+	9250 4350 9050 4350
+Wire Wire Line
+	9050 4350 9050 4300
 $EndSCHEMATC
